File: HW/Robot/Servo_Current_Limiter/Servo_Current_Limiter.kicad_pcb (KiCad board)
At the start: 2 copper layers, 96.5 x 48.3 mm, 55 parts, among them J1 1x2 2.54mm male, J11 1x2 2.54mm male, J2 1x5 2.54mm 90deg female, J5 1x8 2.54mm 90deg male, J6 1x6 2.54mm 90deg female, J9 2x2 2.54mm male, Q1 BC639, Q2 BC639, Q3 BC639, Q4 BC547, Q5 IRF9Z34N, Q6 IRF9Z34N, SW1 PB, SW2 PB, SW3 PB, SW4 PB, SW5 PB, SW6 PB

Commit message: Now finished.
Parts:
- removed D1, D10, D13, D16, D4, D7: Red 5mm, For_Rasterboard:LED_D3.0mm_Pinf
- removed D11, D14, D17, D2, D5, D8: Yellow 5mm, For_Rasterboard:LED_D3.0mm_Pinf
- removed D12, D15, D18, D3, D6, D9: Green 5mm, For_Rasterboard:LED_D3.0mm_Pinf
- removed J5: 1x8 2.54mm 90deg male, Connector_PinHeader_2.54mm:PinHeader_1x09_P2.54mm_Horizontal
- removed J6: 1x6 2.54mm 90deg female, Connector_PinSocket_2.54mm:PinSocket_1x06_P2.54mm_Horizontal
- removed J9: 2x2 2.54mm male, Connector_PinHeader_2.54mm:PinHeader_2x02_P2.54mm_Vertical
- removed JP1, JP2: 1x2 2.54mm male, Connector_PinHeader_2.54mm:PinHeader_1x02_P2.54mm_Vertical
- removed Q3: BC639, For_Rasterboard:TO-92_Inline_inf
- removed Q4: BC547, For_Rasterboard:TO-92_Inline_inf
- removed Q5, Q6: IRF9Z34N, Package_TO_SOT_THT:TO-220-3_Vertical
- removed R10: 4k7, Resistor_THT:R_Axial_DIN0207_L6.3mm_D2.5mm_P7.62mm_Horizontal
- removed R11: 1k, Resistor_THT:R_Axial_DIN0207_L6.3mm_D2.5mm_P10.16mm_Horizontal
- removed R12: 10k, Resistor_THT:R_Axial_DIN0207_L6.3mm_D2.5mm_P5.08mm_Vertical
- removed R13: 10k, Resistor_THT:R_Axial_DIN0204_L3.6mm_D1.6mm_P2.54mm_Vertical
- removed R14: 10k, For_Rasterboard:R_Axial_DIN0207_L6.3mm_D2.5mm_P2.54mm_Vertical
- removed R15: 100, For_Rasterboard:R_Axial_DIN0207_L6.3mm_D2.5mm_Pinf_Horizontal
- removed R8, R9: 1k, For_Rasterboard:R_Axial_DIN0207_L6.3mm_D2.5mm_Pinf_Horizontal
- removed SW1, SW2, SW3, SW4, SW5, SW6: PB, For_Rasterboard:SW_PUSH_5mm
- added C2: 100n, For_Rasterboard:C_Disc_D3.0mm_W1.6mm_Pinf, F.Cu at (188.4, 113.3)
- added J3: 1x1 2.54mm male, Connector_PinHeader_2.54mm:PinHeader_1x01_P2.54mm_Vertical, F.Cu at (191.2, 125.9)
- added RV1: 250, Potentiometer_THT:Potentiometer_Piher_PT-10-V10_Vertical, F.Cu at (147.1, 108.6)
- added RV2: 100k, Potentiometer_THT:Potentiometer_Piher_PT-10-H01_Horizontal, F.Cu at (180.1, 103.5)
- added U1: TL071, Package_DIP:DIP-8_W7.62mm, F.Cu at (187.3, 102.1)
- C1: footprint For_Rasterboard:C_Disc_D3.0mm_W1.6mm_P2.50mm -> For_Rasterboard:C_Disc_D3.0mm_W1.6mm_Pinf
- J1: value 1x2 2.54mm male -> 1x1 2.54mm male; footprint Extra_Common:MOLEX-22-23-2021 -> Connector_PinHeader_2.54mm:PinHeader_1x01_P2.54mm_Vertical
- J2: value 1x5 2.54mm 90deg female -> 1x5 2.54mm male; footprint Connector_PinSocket_2.54mm:PinSocket_1x05_P2.54mm_Horizontal -> Connector_PinSocket_2.54mm:PinSocket_1x05_P2.54mm_Vertical
- Q1: value BC639 -> IRF4905; footprint For_Rasterboard:TO-92_Inline_inf -> Package_TO_SOT_THT:TO-220-3_Vertical
- Q2: value BC639 -> BC338
- R1: value 100 -> 220
- R2: value 100 -> 0.1; footprint For_Rasterboard:R_Axial_DIN0207_L6.3mm_D2.5mm_Pinf_Horizontal -> Resistor_THT:R_Axial_DIN0207_L6.3mm_D2.5mm_P10.16mm_Horizontal
- R3, R6: value 100 -> 220k
- R4, R5: value 100 -> 220k; footprint For_Rasterboard:R_Axial_DIN0207_L6.3mm_D2.5mm_Pinf_Horizontal -> For_Rasterboard:R_Axial_DIN0207_L6.3mm_D2.5mm_P7.62mm_Horizontal
- R7: value 1k -> 1k5; footprint For_Rasterboard:R_Axial_DIN0207_L6.3mm_D2.5mm_Pinf_Horizontal -> For_Rasterboard:R_Axial_DIN0207_L6.3mm_D2.5mm_P5.08mm_Vertical
- moved C1 77.7 mm to (198.1, 101.6), turned to 0 degrees
- moved R6 77.2 mm to (179.7, 125.6)
- moved R4 69.1 mm to (179.7, 129.7)
- moved J11 66.3 mm to (144.1, 126.7), turned to 0 degrees
- moved Q2 64.8 mm to (160.6, 109.2)
- moved R3 64.8 mm to (190.5, 121.5)
- moved R5 60.3 mm to (179.7, 121.5)
- moved R1 57.5 mm to (155.4, 113.9)
- moved R7 55.0 mm to (180.2, 114.0)
- moved R2 43.8 mm to (142.1, 116.8)
- moved J1 35.3 mm to (166.9, 114.1), turned to 0 degrees
- moved Q1 26.1 mm to (162.3, 104.0)
- moved J2 16.1 mm to (142.8, 102.3)
Connections:
- A1 pad 10: /COL1 -> unconnected-(A1-Pad10)
- A1 pad 11: /COL2 -> unconnected-(A1-Pad11)
- A1 pad 12: /PB1 -> unconnected-(A1-Pad12)
- A1 pad 13: /PB0 -> unconnected-(A1-Pad13)
- A1 pad 14: /ADC -> unconnected-(A1-Pad14)
- A1 pad 15: /ARD_RX -> unconnected-(A1-Pad15)
- A1 pad 16: /ARD_TX -> unconnected-(A1-Pad16)
- A1 pad 17: /LED0 -> /DIS0
- A1 pad 18: /LED1 -> unconnected-(A1-Pad18)
- A1 pad 19: /LED2 -> unconnected-(A1-Pad19)
- A1 pad 20: /LED3 -> unconnected-(A1-Pad20)
- A1 pad 21: /LED4 -> unconnected-(A1-Pad21)
- A1 pad 22: /LED5 -> unconnected-(A1-Pad22)
- A1 pad 23: /N_RST -> unconnected-(A1-Pad23)
- A1 pad 24: /DTR_SOFT_RST -> unconnected-(A1-Pad24)
- A1 pad 25: /SW_UART_TX -> unconnected-(A1-Pad25)
- A1 pad 26: /N_EN_5V -> unconnected-(A1-Pad26)
- A1 pad 27: /EN_24V -> unconnected-(A1-Pad27)
- A1 pad 9: /COL0 -> /OUT0
- C1 pad 1: /DTR_SOFT_RST -> +5V
- C1 pad 2: /DTR -> GNDA
- J1 pad 1: +24V -> Net-(J1-Pad1)
- J2 pad 2: GND -> unconnected-(J2-Pad2)
- J2 pad 3: /SW_UART_TX -> /ch0/PWM
- J2 pad 4: unconnected-(J2-Pad4) -> /ch0/N
- J2 pad 5: unconnected-(J2-Pad5) -> GND
- Q1 pad 1: GND -> /DIS0
- Q1 pad 2: /led_pb.kicad_sch/N_GREEN -> /ch0/P
- Q1 pad 3: Net-(Q1-Pad3) -> +5V
- Q2 pad 1: GND -> /DIS0
- Q2 pad 2: /led_pb.kicad_sch/N_YELLOW -> /OUT0
- Q2 pad 3: Net-(Q2-Pad3) -> Net-(J1-Pad1)
- R1 pad 1: /LED5 -> +5V
- R2 pad 1: /LED4 -> /ch0/N
- R2 pad 2: Net-(D4-Pad2) -> /ch0/P
- R3 pad 1: /LED3 -> GNDA
- R3 pad 2: Net-(D7-Pad2) -> /ch0/sub/op/IN+
- R4 pad 1: /LED2 -> /ch0/N
- R4 pad 2: Net-(D10-Pad2) -> /ch0/sub/op/IN+
- R5 pad 1: /LED1 -> /ch0/sub/op/IN-
- R5 pad 2: Net-(D13-Pad2) -> /ch0/P
- R6 pad 1: /LED0 -> /OUT0
- R6 pad 2: Net-(D16-Pad2) -> /ch0/sub/op/IN-
- R7 pad 1: /COL2 -> Net-(R7-Pad1)
- R7 pad 2: Net-(Q1-Pad3) -> GND
Routing:
- net /PB0: track 256.5 -> 0.00 mm, vias 22 -> 0
- net /led_pb.kicad_sch/N_GREEN: track 180.3 -> 0.00 mm, vias 8 -> 0
- net (no net): track 180.3 -> 0.00 mm, vias 9 -> 0
- net GND: track 121.9 -> 0.00 mm, vias 13 -> 0
- net /24V: track 33.0 -> 0.00 mm, vias 1 -> 0
- net /UART_FROM_DONGLE: track 31.5 -> 0.00 mm, vias 4 -> 0
- net /UART_RETURN: track 27.9 -> 0.00 mm
- net +24V: track 27.9 -> 0.00 mm
- net /LED0: track 25.4 -> 0.00 mm, vias 1 -> 0
- net /led_pb.kicad_sch/N_YELLOW: track 25.4 -> 0.00 mm, vias 1 -> 0
- net +5V: track 22.9 -> 0.00 mm, vias 2 -> 0
- net /UART_TO_HARNESS: track 20.3 -> 0.00 mm, vias 2 -> 0
- net Net-(D7-Pad2): track 17.8 -> 0.00 mm, vias 2 -> 0
- net unconnected-(J2-Pad5): track 17.8 -> 0.00 mm, vias 2 -> 0
- net Net-(D4-Pad2): track 17.8 -> 0.00 mm, vias 2 -> 0
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Other:
- board outline removed
