File: HW/Robot/Servo_Current_Limiter/Servo_Current_Limiter.kicad_sch (KiCad schematic)
At the start: 7 parts, among them J11 1x2 2.54mm male, J9 2x2 2.54mm male

Commit message: Finished one circuit.
Parts:
- removed C1: 100n, For_Rasterboard:C_Disc_D3.0mm_W1.6mm_P2.50mm, symbol Device:C
- removed J9: 2x2 2.54mm male, Connector_PinHeader_2.54mm:PinHeader_2x02_P2.54mm_Vertical, symbol Connector_Generic:Conn_02x02_Odd_Even
- removed JP1: 1x2 2.54mm male, Connector_PinHeader_2.54mm:PinHeader_1x02_P2.54mm_Vertical, symbol Jumper:Jumper_2_Open
- removed R10: 4k7, Resistor_THT:R_Axial_DIN0207_L6.3mm_D2.5mm_P7.62mm_Horizontal, symbol Device:R
- removed R11: 1k, Resistor_THT:R_Axial_DIN0207_L6.3mm_D2.5mm_P10.16mm_Horizontal, symbol Device:R
Connections:
- net N_RST: no longer A1.23 (D8)
- net ADC: no longer names the net of A1.14 (SCL/A5)
- net ARD_RX: no longer names the net of A1.15 (D0/RX)
- net ARD_TX: no longer names the net of A1.16 (D1/TX)
- net COL0 renamed OUT0
- net COL1: no longer names the net of A1.10 (A1)
- net COL2: no longer names the net of A1.11 (A2)
- net DTR_SOFT_RST: no longer names the net of A1.24 (D9)
- net EN_24V: no longer names the net of A1.27 (D12)
- net LED0 renamed DIS0
- net LED1: no longer names the net of A1.18 (D3)
- net LED2: no longer names the net of A1.19 (D4)
- net LED3: no longer names the net of A1.20 (D5)
- net LED4: no longer names the net of A1.21 (D6)
- net LED5: no longer names the net of A1.22 (D7)
- net N_EN_5V: no longer names the net of A1.26 (D11)
- net PB0: no longer names the net of A1.13 (SDA/A4)
- net PB1: no longer names the net of A1.12 (A3)
- net SW_UART_TX: no longer names the net of A1.25 (D10)
- no-connect marks 8 -> 7
Other:
- sheet ch0 ports: added DISABLE, OUT; removed none
- note removed: "From dongle: 5V GND RXD TXD 3V3"
- moved on the sheet: A1
