File: HW/Robot/Servo_Current_Limiter/channel.kicad_sch (KiCad schematic)
At the start: 8 parts

Commit message: Finished one circuit.
Parts:
- removed Q?: BC547, For_Rasterboard:TO-92_Inline_inf, symbol Transistor_BJT:BC547
- removed Q?: IRF9Z34N, Package_TO_SOT_THT:TO-220-3_Vertical, symbol Device:Q_PMOS_GDS
- removed R?: 10k, Resistor_THT:R_Axial_DIN0207_L6.3mm_D2.5mm_P5.08mm_Vertical, symbol Device:R
- removed R?: 10k, For_Rasterboard:R_Axial_DIN0207_L6.3mm_D2.5mm_P2.54mm_Vertical, symbol Device:R
- removed R?: 10k, Resistor_THT:R_Axial_DIN0204_L3.6mm_D1.6mm_P2.54mm_Vertical, symbol Device:R
- added J?: 1x1 2.54mm male, Connector_PinHeader_2.54mm:PinHeader_1x01_P2.54mm_Vertical, symbol Connector:TestPoint
- added Q?: BC338, Package_TO_SOT_THT:TO-92_Inline, symbol Servo_Current_Limiter-cache:BC338
- added R?: 0.1, Resistor_THT:R_Axial_DIN0207_L6.3mm_D2.5mm_P10.16mm_Horizontal, symbol Device:R
- added RV?: 250, symbol Device:R_Potentiometer
- Q?: value IRF9Z34N -> IRF4905
- R?: value 100 -> 1k
Connections:
- net +5V: now also R?.1
- net GND: now also RV?.3; no longer R?.2
- net 5V renamed N
- net N: now also R?.1; no longer Q?.2 (D)
- net N_EN_5V renamed DISABLE
- net DISABLE: now also Q?.1 (C); no longer R?.1
- new net: J?.1, Q?.3 (E), RV?.2
- new net: R?.2, RV?.1
- new net OUT: Q?.2 (B)
- new net P: Q?.2 (D), R?.2
Other:
- added sheet sub (substracter.kicad_sch)
- moved on the sheet: J?, Q?, R?

Commit message: Now finished.
Parts:
- Q2: renamed from Q?; footprint Package_TO_SOT_THT:TO-92_Inline -> For_Rasterboard:TO-92_Inline_inf
- R1: renamed from R?; value 1k -> 220
- RV1: renamed from RV?; footprint (none) -> Potentiometer_THT:Potentiometer_Piher_PT-10-V10_Vertical
- gave numbers to parts that had none: 4
Changed lines of the file:
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@@
   (symbol (lib_id "power:+5V") (at 140.97 66.04 0) (unit 1)
     (in_bom yes) (on_board yes) (fields_autoplaced)
-    (property "Reference" "#PWR?" (id 0) (at 140.97 69.85 0)
+    (property "Reference" "#PWR01" (id 0) (at 140.97 69.85 0)
       (effects (font (size 1.27 1.27)) hide)
     )
@@
   (symbol (lib_id "power:+5V") (at 168.91 41.91 90) (unit 1)
     (in_bom yes) (on_board yes)
-    (property "Reference" "#PWR?" (id 0) (at 172.72 41.91 0)
+    (property "Reference" "#PWR05" (id 0) (at 172.72 41.91 0)
       (effects (font (size 1.27 1.27)) hide)
     )
@@
   (symbol (lib_id "Connector:TestPoint") (at 160.02 80.01 0) (unit 1)
     (in_bom yes) (on_board yes)
-    (property "Reference" "J?" (id 0) (at 160.02 71.12 0))
+    (property "Reference" "J1" (id 0) (at 160.02 71.12 0))
     (property "Value" "1x1 2.54mm male" (id 1) (at 160.02 73.66 0))
     (property "Footprint" "Connector_PinHeader_2.54mm:PinHeader_1x01_P2.54mm_Vertical" (id 2) (at 160.02 80.01 0)
@@
   (symbol (lib_id "Device:R") (at 140.97 72.39 0) (unit 1)
     (in_bom yes) (on_board yes)
-    (property "Reference" "R?" (id 0) (at 135.7122 72.39 90))
-    (property "Value" "1k" (id 1) (at 138.0236 72.39 90))
+    (property "Reference" "R1" (id 0) (at 135.7122 72.39 90))
+    (property "Value" "220" (id 1) (at 138.0236 72.39 90))
     (property "Footprint" "For_Rasterboard:R_Axial_DIN0207_L6.3mm_D2.5mm_Pinf_Horizontal" (id 2) (at 139.192 72.39 90)
       (effects (font (size 1.27 1.27)) hide)
@@
   (symbol (lib_id "Device:Q_PMOS_GDS") (at 177.8 44.45 270) (mirror x) (unit 1)
     (in_bom yes) (on_board yes)
-    (property "Reference" "Q?" (id 0) (at 177.8 35.7632 90))
+    (property "Reference" "Q1" (id 0) (at 177.8 35.7632 90))
     (property "Value" "IRF4905" (id 1) (at 177.8 38.0746 90))
     (property "Footprint" "Package_TO_SOT_THT:TO-220-3_Vertical" (id 2) (at 180.34 39.37 0)
@@
   (symbol (lib_id "Servo_Current_Limiter-cache:BC338") (at 180.34 77.47 0) (mirror y) (unit 1)
     (in_bom yes) (on_board yes) (fields_autoplaced)
-    (property "Reference" "Q?" (id 0) (at 175.26 76.1999 0)
+    (property "Reference" "Q2" (id 0) (at 175.26 76.1999 0)
       (effects (font (size 1.27 1.27)) (justify left))
     )
@@
       (effects (font (size 1.27 1.27)) (justify left))
     )
-    (property "Footprint" "Package_TO_SOT_THT:TO-92_Inline" (id 2) (at 175.26 79.375 0)
+    (property "Footprint" "For_Rasterboard:TO-92_Inline_inf" (id 2) (at 175.26 79.375 0)
       (effects (font (size 1.27 1.27) italic) (justify left) hide)
     )
@@
   (symbol (lib_id "power:GND") (at 140.97 90.17 0) (mirror y) (unit 1)
     (in_bom yes) (on_board yes)
-    (property "Reference" "#PWR?" (id 0) (at 140.97 96.52 0)
+    (property "Reference" "#PWR04" (id 0) (at 140.97 96.52 0)
       (effects (font (size 1.27 1.27)) hide)
     )
@@
   (symbol (lib_id "Device:R_Potentiometer") (at 140.97 82.55 0) (unit 1)
     (in_bom yes) (on_board yes) (fields_autoplaced)
-    (property "Reference" "RV?" (id 0) (at 138.43 81.2799 0)
+    (property "Reference" "RV1" (id 0) (at 138.43 81.2799 0)
       (effects (font (size 1.27 1.27)) (justify right))
     )
@@
       (effects (font (size 1.27 1.27)) (justify right))
     )
-    (property "Footprint" "" (id 2) (at 140.97 82.55 0)
+    (property "Footprint" "Potentiometer_THT:Potentiometer_Piher_PT-10-V10_Vertical" (id 2) (at 140.97 82.55 0)
       (effects (font (size 1.27 1.27)) hide)
     )
@@
   (symbol (lib_id "Device:R") (at 191.77 41.91 270) (unit 1)
     (in_bom yes) (on_board yes)
-    (property "Reference" "R?" (id 0) (at 191.77 36.6522 90))
+    (property "Reference" "R2" (id 0) (at 191.77 36.6522 90))
     (property "Value" "0.1" (id 1) (at 191.77 38.9636 90))
     (property "Footprint" "Resistor_THT:R_Axial_DIN0207_L6.3mm_D2.5mm_P10.16mm_Horizontal" (id 2) (at 191.77 40.132 90)
@@
   (symbol (lib_id "power:GND") (at 231.775 53.34 270) (unit 1)
     (in_bom yes) (on_board yes) (fields_autoplaced)
-    (property "Reference" "#PWR?" (id 0) (at 225.425 53.34 0)
+    (property "Reference" "#PWR06" (id 0) (at 225.425 53.34 0)
       (effects (font (size 1.27 1.27)) hide)
     )
@@
   (symbol (lib_id "Connector_Generic:Conn_01x05") (at 238.76 48.26 0) (unit 1)
     (in_bom yes) (on_board yes)
-    (property "Reference" "J?" (id 0) (at 236.22 39.37 0)
+    (property "Reference" "J2" (id 0) (at 236.22 39.37 0)
       (effects (font (size 1.27 1.27)) (justify left))
     )
