File: HW/Robot/Servo_Current_Limiter/op_amp.kicad_sch (KiCad schematic)
At the start: 5 parts

Commit message: Now finished.
Parts:
- gave numbers to parts that had none: 5
Changed lines of the file:
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@@
   (symbol (lib_id "power:GNDA") (at 133.35 59.69 270) (unit 1)
     (in_bom yes) (on_board yes) (fields_autoplaced)
-    (property "Reference" "#PWR?" (id 0) (at 127 59.69 0)
+    (property "Reference" "#PWR010" (id 0) (at 127 59.69 0)
       (effects (font (size 1.27 1.27)) hide)
     )
@@
   (symbol (lib_id "power:+5V") (at 143.51 52.07 0) (unit 1)
     (in_bom yes) (on_board yes) (fields_autoplaced)
-    (property "Reference" "#PWR?" (id 0) (at 143.51 55.88 0)
+    (property "Reference" "#PWR012" (id 0) (at 143.51 55.88 0)
       (effects (font (size 1.27 1.27)) hide)
     )
@@
   (symbol (lib_id "power:GND") (at 143.51 88.9 0) (unit 1)
     (in_bom yes) (on_board yes) (fields_autoplaced)
-    (property "Reference" "#PWR?" (id 0) (at 143.51 95.25 0)
+    (property "Reference" "#PWR013" (id 0) (at 143.51 95.25 0)
       (effects (font (size 1.27 1.27)) hide)
     )
@@
   (symbol (lib_id "power:GNDA") (at 133.35 87.63 270) (unit 1)
     (in_bom yes) (on_board yes) (fields_autoplaced)
-    (property "Reference" "#PWR?" (id 0) (at 127 87.63 0)
+    (property "Reference" "#PWR011" (id 0) (at 127 87.63 0)
       (effects (font (size 1.27 1.27)) hide)
     )
@@
   (symbol (lib_id "Device:C") (at 139.7 59.69 270) (unit 1)
     (in_bom yes) (on_board yes) (fields_autoplaced)
-    (property "Reference" "C?" (id 0) (at 139.7 52.07 90))
+    (property "Reference" "C1" (id 0) (at 139.7 52.07 90))
     (property "Value" "100n" (id 1) (at 139.7 54.61 90))
     (property "Footprint" "For_Rasterboard:C_Disc_D3.0mm_W1.6mm_Pinf" (id 2) (at 135.89 60.6552 0)
@@
   (symbol (lib_id "Device:R") (at 149.86 97.79 0) (unit 1)
     (in_bom yes) (on_board yes) (fields_autoplaced)
-    (property "Reference" "R?" (id 0) (at 152.4 96.5199 0)
+    (property "Reference" "R7" (id 0) (at 152.4 96.5199 0)
       (effects (font (size 1.27 1.27)) (justify left))
     )
@@
   (symbol (lib_id "Device:C") (at 139.7 87.63 270) (unit 1)
     (in_bom yes) (on_board yes) (fields_autoplaced)
-    (property "Reference" "C?" (id 0) (at 139.7 80.01 90))
+    (property "Reference" "C2" (id 0) (at 139.7 80.01 90))
     (property "Value" "100n" (id 1) (at 139.7 82.55 90))
     (property "Footprint" "For_Rasterboard:C_Disc_D3.0mm_W1.6mm_Pinf" (id 2) (at 135.89 88.5952 0)
@@
   (symbol (lib_id "power:GND") (at 149.86 104.14 0) (unit 1)
     (in_bom yes) (on_board yes) (fields_autoplaced)
-    (property "Reference" "#PWR?" (id 0) (at 149.86 110.49 0)
+    (property "Reference" "#PWR014" (id 0) (at 149.86 110.49 0)
       (effects (font (size 1.27 1.27)) hide)
     )
@@
   (symbol (lib_id "Device:R_Potentiometer_Trim") (at 149.86 87.63 270) (unit 1)
     (in_bom yes) (on_board yes) (fields_autoplaced)
-    (property "Reference" "RV?" (id 0) (at 149.86 81.28 90))
+    (property "Reference" "RV2" (id 0) (at 149.86 81.28 90))
     (property "Value" "100k" (id 1) (at 149.86 83.82 90))
     (property "Footprint" "Potentiometer_THT:Potentiometer_Piher_PT-10-H01_Horizontal" (id 2) (at 149.86 87.63 0)
@@
   (symbol (lib_id "Amplifier_Operational:TL071") (at 146.05 71.12 0) (unit 1)
     (in_bom yes) (on_board yes) (fields_autoplaced)
-    (property "Reference" "U?" (id 0) (at 154.94 66.421 0))
+    (property "Reference" "U1" (id 0) (at 154.94 66.421 0))
     (property "Value" "TL071" (id 1) (at 154.94 68.961 0))
     (property "Footprint" "Package_DIP:DIP-8_W7.62mm" (id 2) (at 147.32 69.85 0)
