File: HW/Robot/Servo_Current_Limiter/substracter.kicad_sch (KiCad schematic)
At the start: 5 parts

Commit message: Now finished.
Parts:
- gave numbers to parts that had none: 5
Changed lines of the file:
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@@
   (symbol (lib_id "Connector:TestPoint") (at 207.01 78.74 0) (unit 1)
     (in_bom yes) (on_board yes)
-    (property "Reference" "J?" (id 0) (at 207.01 69.85 0))
+    (property "Reference" "J3" (id 0) (at 207.01 69.85 0))
     (property "Value" "1x1 2.54mm male" (id 1) (at 207.01 72.39 0))
     (property "Footprint" "Connector_PinHeader_2.54mm:PinHeader_1x01_P2.54mm_Vertical" (id 2) (at 207.01 78.74 0)
@@
   (symbol (lib_id "power:GNDA") (at 132.08 71.12 270) (unit 1)
     (in_bom yes) (on_board yes) (fields_autoplaced)
-    (property "Reference" "#PWR?" (id 0) (at 125.73 71.12 0)
+    (property "Reference" "#PWR07" (id 0) (at 125.73 71.12 0)
       (effects (font (size 1.27 1.27)) hide)
     )
@@
   (symbol (lib_id "Device:R") (at 146.05 83.82 270) (mirror x) (unit 1)
     (in_bom yes) (on_board yes)
-    (property "Reference" "R?" (id 0) (at 146.05 89.0778 90))
+    (property "Reference" "R5" (id 0) (at 146.05 89.0778 90))
     (property "Value" "220k" (id 1) (at 146.05 86.7664 90))
     (property "Footprint" "For_Rasterboard:R_Axial_DIN0207_L6.3mm_D2.5mm_P7.62mm_Horizontal" (id 2) (at 146.05 85.598 90)
@@
   (symbol (lib_id "Device:R") (at 167.64 99.06 270) (unit 1)
     (in_bom yes) (on_board yes)
-    (property "Reference" "R?" (id 0) (at 167.64 93.8022 90))
+    (property "Reference" "R6" (id 0) (at 167.64 93.8022 90))
     (property "Value" "220k" (id 1) (at 167.64 96.1136 90))
     (property "Footprint" "For_Rasterboard:R_Axial_DIN0207_L6.3mm_D2.5mm_Pinf_Horizontal" (id 2) (at 167.64 97.282 90)
@@
   (symbol (lib_id "Device:R") (at 146.05 71.12 90) (mirror x) (unit 1)
     (in_bom yes) (on_board yes)
-    (property "Reference" "R?" (id 0) (at 146.05 65.8622 90))
+    (property "Reference" "R3" (id 0) (at 146.05 65.8622 90))
     (property "Value" "220k" (id 1) (at 146.05 68.1736 90))
     (property "Footprint" "For_Rasterboard:R_Axial_DIN0207_L6.3mm_D2.5mm_Pinf_Horizontal" (id 2) (at 146.05 69.342 90)
@@
   (symbol (lib_id "Device:R") (at 146.05 78.74 90) (mirror x) (unit 1)
     (in_bom yes) (on_board yes)
-    (property "Reference" "R?" (id 0) (at 146.05 73.4822 90))
+    (property "Reference" "R4" (id 0) (at 146.05 73.4822 90))
     (property "Value" "220k" (id 1) (at 146.05 75.7936 90))
     (property "Footprint" "For_Rasterboard:R_Axial_DIN0207_L6.3mm_D2.5mm_P7.62mm_Horizontal" (id 2) (at 146.05 76.962 90)
