File: HW/IoT/Tuzibaba_RFID/channel.kicad_sch (KiCad schematic)
At the start: 7 parts, among them J1 1x1 2.54mm male, J2 1x5 2.54mm male, Q1 IRF4905, Q2 BC338

Commit message: Clear repository of irrelevant directories and files
Parts:
- Q2: symbol Servo_Current_Limiter-cache:BC338 -> Tuzibaba-cache:BC338
Changed lines of the file:
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@@
     (pin "3")
   )
-  (symbol (lib_id "Servo_Current_Limiter-cache:BC338") (at 180.34 77.47 0) (mirror y) (unit 1)
+  (symbol (lib_id "Tuzibaba-cache:BC338") (at 180.34 77.47 0) (mirror y) (unit 1)
     (in_bom yes) (on_board yes) (fields_autoplaced)
     (property "Reference" "Q2" (id 0) (at 175.26 76.1999 0)
